File: hardware/sablier/sablier.kicad_pcb (KiCad board)
At the start: 2 copper layers, 57.1 x 50.6 mm, 5 parts, among them J1 CX70M-24P1

Commit message: PCB mechanical validation
Parts:
- removed the REF** at (151.6, 104.1)
- added G***: LOGO, 0_stimulu-common:sinestimulus_logo, F.Cu at (151.6, 113.1)
- added M1: vibrating_motor_adafruit, 0_stimulu-common:vibrating_motor_adafruit, F.Cu at (151.6, 104.1)
- added REF**: order_number, 0_stimulu-common:order_number, F.Cu at (151.6, 104.1)
Routing:
- net (no net): track 79.2 -> 49.8 mm, vias 2 -> 0
- net Net-(J1-PadSH): track 9.06 -> 0.00 mm
- added copper zone on B.Cu, net Net-(J1-PadSH)
- added copper zone on F.Cu, net Net-(J1-PadSH)
Other:
- board text added: "190509 REV 1"
- board text added: "SABLIER mechanical validation"
